File: pcb/stm32-usb-ble-devkit.sch (EAGLE design)
At the start: 98 parts, among them CN1 USB-MICROB-2TABS, CN2 USB-C-2.0-FEMALE, CN3 USB-C-2.0-FEMALE, Q2 AO3402, Q4 AO3401, Q6 AO3401, Q8 AO3401, U1 STM32F103-48LQFP, U2 STM32F205-64, U3 TUSB320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

Commit message: pcb: Replace PSU 0805 caps with 0603
Parts:
- C18, C19, C20, C21: device tuetuopay:C0805 -> tuetuopay:C0603
Changed lines of the file:
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@@
 <part name="+3V23" library="supply1" library_urn="urn:adsk.eagle:library:371" deviceset="+3V3" device=""/>
 <part name="U6" library="tuetuopay" deviceset="LDO" device="AMS1117" value="AMS1117-3.3"/>
-<part name="C18" library="tuetuopay" deviceset="C" device="0805" value="22u"/>
-<part name="C19" library="tuetuopay" deviceset="C" device="0805" value="22u"/>
+<part name="C18" library="tuetuopay" deviceset="C" device="0603" value="22u"/>
+<part name="C19" library="tuetuopay" deviceset="C" device="0603" value="22u"/>
 <part name="GND33" library="supply1" library_urn="urn:adsk.eagle:library:371" deviceset="GND" device=""/>
 <part name="+3V24" library="supply1" library_urn="urn:adsk.eagle:library:371" deviceset="+3V3" device=""/>
@@
 <part name="JP13" library="pinhead" library_urn="urn:adsk.eagle:library:325" deviceset="PINHD-2X3" device="" package3d_urn="urn:adsk.eagle:package:22462/2"/>
 <part name="TP13" library="testpad" library_urn="urn:adsk.eagle:library:385" deviceset="PTR1" device="B1,27" package3d_urn="urn:adsk.eagle:package:27944/1"/>
-<part name="C20" library="tuetuopay" deviceset="C" device="0805" value="100n"/>
-<part name="C21" library="tuetuopay" deviceset="C" device="0805" value="100n"/>
+<part name="C20" library="tuetuopay" deviceset="C" device="0603" value="100n"/>
+<part name="C21" library="tuetuopay" deviceset="C" device="0603" value="100n"/>
 <part name="R17" library="tuetuopay" deviceset="R" device="R0603" value="100k"/>
 <part name="R19" library="tuetuopay" deviceset="R" device="R0603" value="100k"/>
